File: KiCAD/music_box.sch (KiCad schematic (older format))
At the start: 38 parts, among them Q1 2N3904, SW1 power, SW2 mode, SW3 play, U1 LM3940-3.3, U2 EFM8BB10F8G_SOIC16, U3 LM386

Commit message: modification schématique, R10 avait la mauvaise valeur.
Parts:
- R10: value 15K -> 3K
Changed lines of the file:
@@
 LIBS:valves
 LIBS:librairie-personnelle
+LIBS:music_box-cache
 EELAYER 25 0
 EELAYER END
@@
 P 7150 4200
 F 0 "R10" V 7230 4200 50  0000 C CNN
-F 1 "15K" V 7150 4200 50  0000 C CNN
+F 1 "3K" V 7150 4200 50  0000 C CNN
 F 2 "" V 7080 4200 50  0000 C CNN
 F 3 "" H 7150 4200 50  0000 C CNN
